File: rc65xx/overview_65xx.kicad_sch (KiCad schematic)
At the start: 198 parts, among them J101 ABORT, J102 Sync/VPA, J103 SO/MX, J104 ABORT, J105 Cx, J106 CF Card, J107 Barrel_Jack, J108 DE9_Plug_MountingHoles, J109 Conn_01x08, J110 DE9_Plug_MountingHoles, J111 Conn_01x08, J112 P1B, J113 P2B, J114 P2A, J115 P3A, J116 P3B, J117 Conn_02x20_Odd_Even, J118 Conn_02x22_Odd_Even, J119 IDE_VCC, J120 Clock_Sel, SW101 SW_SPDT, SW102 RESET, U101 65C02 / 65816, U102 SST39SF040, U103 W65C22SxP, U104 W65C22SxP, U105 6525, U106 6525, U107 6551, U108 W65C22SxP, U109 AS6C4008-55PCN, U110 CY62256-70PC, U111 74HC688, U112 74HC00, U113 74154, U114 74HC04, U115 6520, U116 74HC00, U117 74LS20, U118 74HC138, U119 8580, U120 AS6C4008-55PCN, U121 74HC00, U122 74HCT74, U123 74LS32, U124 74HC00, U125 MAX232, U126 MAX232, U127 MAX232, U128 MAX232, U129 6551, U130 74HC138, U131 74HC00, U132 74AHCT04, U133 74LS393, U134 74HC02, U135 74AHC04, U136 GAL16V8, U137 SA39-11EWA, U138 SA39-11EWA, U139 GAL16V8, U140 SA39-11EWA, U141 GAL16V8, U142 SA39-11EWA, U143 GAL16V8, U144 SA39-11EWA, U145 GAL16V8, U146 SA39-11EWA, U147 GAL16V8, X101 1.8432MHz, X102 8MHz

Commit message: finalize Schematic
Parts:
- removed J102: Sync/VPA, symbol Connector_Generic:Conn_01x03
- removed J104: ABORT, symbol Connector_Generic:Conn_01x03
- removed J112: P1B, symbol Connector_Generic:Conn_01x12
- removed unit 4 of U123
- added BZ101: Buzzer, symbol Device:Buzzer
- added C121, C122: 10µ, symbol Device:C
- added C123, C133: 1µ, symbol Device:C
- added C124, C125, C126, C127, C128, C129, C130, C131, C132, C134, C136: 100n, symbol Device:C
- added C135: 15p, symbol Device:C
- added D120: 1N5817, Diode_THT:D_DO-41_SOD81_P10.16mm_Horizontal, symbol Diode:1N5817
- added D121: USB_EN, symbol Device:LED
- added D122: ACTIV, symbol Device:LED
- added J102: Bus Connector, symbol Connector_Generic:Conn_02x39_Odd_Even
- added J121: USB_C_Receptacle_USB2.0_14P, symbol Connector:USB_C_Receptacle_USB2.0_14P
- added J122: DE15_Receptacle_HighDensity_MountingHoles, symbol Connector:DE15_Receptacle_HighDensity_MountingHoles
- added J123: Keyboard, symbol Connector:USB_A
- added J124: Micro_SD_Card, symbol Connector:Micro_SD_Card
- added J125: IOs, symbol Connector_Generic:Conn_01x09
- added J126: UART, symbol Connector_Generic:Conn_01x04
- added JP106: 0, symbol Jumper:SolderJumper_2_Bridged
- added JP107, JP110, JP112: 1, symbol Jumper:SolderJumper_2_Bridged
- added JP108, JP111, JP113: 2, symbol Jumper:SolderJumper_2_Open
- added JP109: 3, symbol Jumper:SolderJumper_2_Open
- added Q101, Q103, Q104, Q105: BSS138, Package_TO_SOT_SMD:SOT-23, symbol Transistor_FET:BSS138
- added Q102: BSS84, Package_TO_SOT_SMD:SOT-23, symbol Transistor_FET:BSS84
- added R176, R180, R187, R188, R189, R190, R191, R192, R193, R194, R200, R201, R202, R203, R216, R219: 1k, symbol Device:R
- added R177, R181, R213, R214, R215, R217, R221, R222, R223, R224, R225, R226: 10k, symbol Device:R
- added R178, R179: 27R4, symbol Device:R
- added R182, R198, R207: 12k, symbol Device:R
- added R183, R197, R206: 24k, symbol Device:R
- added R184, R185, R186, R195, R196, R199, R204, R205, R208: 2k, symbol Device:R
- added R209, R210: 47, symbol Device:R
- added R211, R212: 5k1, symbol Device:R
- added R218, R220: 470, symbol Device:R
- added RN105: 3k3, Resistor_THT:R_Array_SIP9, symbol Device:R_Network08
- added SW103: BOOTSEL, symbol Switch:SW_SPST
- added SW104: RST, symbol Switch:SW_SPST
- added SW105: T1, symbol Switch:SW_SPST
- added SW106: T2, symbol Switch:SW_SPST
- added SW107: T3, symbol Switch:SW_SPST
- added U148: RP2040, Package_DFN_QFN:QFN-56-1EP_7x7mm_P0.4mm_EP3.2x3.2mm, symbol MCU_RaspberryPi:RP2040
- added U149: AMS1117-3.3, Package_TO_SOT_SMD:SOT-223-3_TabPin2, symbol Regulator_Linear:AMS1117-3.3
- added U150: W25Q128JVS, Package_SO:SOIC-8_5.23x5.23mm_P1.27mm, symbol Memory_Flash:W25Q128JVS
- added U151: PCA9536D, Package_SO:SOIC-8_3.9x4.9mm_P1.27mm, symbol Interface_Expansion:PCA9536D
- added Y101: ABM8-272-T3 12MHZ, symbol Device:Crystal_GND24
Connections:
- net +5V: now also BZ101.1 (+), C122.1, J102.1 (Pin_1), J102.2 (Pin_2), J102.23 (Pin_23), J102.24 (Pin_24), J102.77 (Pin_77), J102.78 (Pin_78), J121.A4 (VBUS), J121.A9 (VBUS), J121.B4 (VBUS), J121.B9 (VBUS), J125.1 (Pin_1), J126.1 (Pin_1), Q102.2 (S), R217.1, R222.1, R224.1, RN105.1 (common), U149.3 (VI)
- net A0: now also J102.3 (Pin_3)
- net A1: now also J102.4 (Pin_4)
- net A10: now also J102.15 (Pin_15)
- net A11: now also J102.16 (Pin_16)
- net A12: now also J102.17 (Pin_17)
- net A13: now also J102.18 (Pin_18)
- net A14: now also J102.21 (Pin_21)
- net A15: now also J102.20 (Pin_20)
- net A2: now also J102.5 (Pin_5)
- net A3: now also J102.6 (Pin_6)
- net A4: now also J102.9 (Pin_9)
- net A5: now also J102.8 (Pin_8)
- net A6: now also J102.11 (Pin_11)
- net A7: now also J102.10 (Pin_10)
- net A8: now also J102.13 (Pin_13)
- net A9: now also J102.12 (Pin_12)
- net ACIA1: now also JP106.2 (B), JP108.1 (A); no longer U130.15 (~{Y0})
- net ACIA2: now also JP107.2 (B), JP109.1 (A); no longer U130.14 (~{Y1})
- net BE: now also J102.70 (Pin_70)
- net CLK: now also J102.73 (Pin_73)
- net D0: now also J102.25 (Pin_25)
- net D1: now also J102.26 (Pin_26)
- net D2: now also J102.27 (Pin_27)
- net D3: now also J102.28 (Pin_28)
- net D4: now also J102.31 (Pin_31)
- net D5: now also J102.32 (Pin_32)
- net D6: now also J102.33 (Pin_33)
- net D7: now also J102.34 (Pin_34)
- net E: now also J102.72 (Pin_72)
- net GND: now also C121.2, C122.2, C123.2, C124.2, C125.2, C126.2, C127.2, C128.2, C129.2, C130.2, C131.2, C132.2, C133.2, C134.2, C135.2, C136.2, D120.2 (A), D121.1 (K), D122.1 (K), J102.14 (Pin_14), J102.19 (Pin_19), J102.22 (Pin_22), J102.29 (Pin_29), J102.30 (Pin_30), J102.35 (Pin_35), J102.36 (Pin_36), J102.53 (Pin_53), J102.54 (Pin_54), J102.59 (Pin_59), J102.60 (Pin_60), J102.65 (Pin_65), J102.66 (Pin_66), J102.7 (Pin_7), J102.71 (Pin_71), J102.74 (Pin_74), J102.75 (Pin_75), J121.A1 (GND), J121.A12 (GND), J121.B1 (GND), J121.B12 (GND), J121.S1 (SHIELD), J122.0, J122.10, J122.5, J122.6, J122.7, J122.8, J123.4 (GND), J123.5 (Shield), J124.6 (VSS), J124.9 (SHIELD), J125.9 (Pin_9), J126.4 (Pin_4), Q101.2 (S), Q103.2 (S), R211.1, R212.1, SW103.1 (A), SW104.1 (A), U148.57 (GND), U149.1 (GND), U150.4 (GND), U151.4 (VSS), Y101.2, Y101.4
- net M/X: now also J102.76 (Pin_76)
- net PAGE: now also J102.51 (Pin_51)
- net PORT_112: now also U124.2
- net PORT_192: no longer U124.1
- net PORT_208: no longer U124.2
- net PORT_96: now also U124.1
- net RDY: now also J102.68 (Pin_68)
- net R/~{W}: now also J102.69 (Pin_69)
- net ~{H_RAM}: now also J102.57 (Pin_57)
- net ~{IO}: now also J102.58 (Pin_58)
- net ~{IRQ_0}: now also U104.21 (~{IRQ}), J102.47 (Pin_47); no longer U107.26 (~{IRQ})
- net ~{IRQ_1}: now also U108.21 (~{IRQ}), J102.45 (Pin_45); no longer U129.26 (~{IRQ})
- net ~{IRQ_2}: now also U103.21 (~{IRQ}), J102.43 (Pin_43); no longer U108.21 (~{IRQ})
- net ~{IRQ_3}: now also J102.41 (Pin_41); no longer U103.21 (~{IRQ})
- net ~{IRQ_4}: now also J102.39 (Pin_39)
- net ~{IRQ}: now also J102.37 (Pin_37)
- net ~{L_RAM}: now also J102.55 (Pin_55)
- net ~{ML}: now also J102.63 (Pin_63)
- net ~{NMI}: now also J102.49 (Pin_49)
- net ~{RES}: now also J102.67 (Pin_67)
- net ~{ROM}: now also J102.56 (Pin_56)
- net ~{VP}: now also J102.61 (Pin_61)
- net P2/VDA: now reaches U101.39 (ϕ2)
- net P2/VDA: now also J102.64 (Pin_64)
- net SYNC/VPA: now reaches U101.7 (SYNC)
- net SYNC/VPA: now also J102.62 (Pin_62)
- net at J106.35 (Pin_35): now also U123.8
- net ~{IRQ_0.0}: now reaches U104.10 (PB0)
- net ~{IRQ_0.0}: now also J102.52 (Pin_52), JP110.1 (A), RN105.2 (R1)
- net ~{IRQ_0.1}: now reaches U104.11 (PB1)
- net ~{IRQ_0.1}: now also J102.50 (Pin_50), JP112.1 (A), RN105.3 (R2)
- net ~{IRQ_0.2}: now reaches U104.12 (PB2)
- net ~{IRQ_0.2}: now also J102.48 (Pin_48), JP111.2 (B), RN105.4 (R3)
- net ~{IRQ_0.3}: now reaches U104.13 (PB3)
- net ~{IRQ_0.3}: now also J102.46 (Pin_46), JP113.2 (B), RN105.5 (R4)
- net ~{IRQ_0.4}: now reaches U104.14 (PB4)
- net ~{IRQ_0.4}: now also J102.44 (Pin_44), RN105.6 (R5)
- net ~{IRQ_0.5}: now reaches U104.15 (PB5)
- net ~{IRQ_0.5}: now also J102.42 (Pin_42), RN105.7 (R6)
- net ~{IRQ_0.6}: now reaches U104.16 (PB6)
- net ~{IRQ_0.6}: now also J102.40 (Pin_40), RN105.8 (R7)
- net ~{IRQ_0.7}: now reaches U104.17 (PB7)
- net ~{IRQ_0.7}: now also J102.38 (Pin_38), RN105.9 (R8)
- net at U130.12 (~{Y3}): now also JP109.2 (B)
- net at U130.13 (~{Y2}): now also JP108.2 (B)
- new net: R178.2, U148.47 (USB_DP)
- new net: J121.A5 (CC1), R212.2
- new net: R191.1, SW106.1 (A)
- new net: R191.2, R197.2, R198.2, U148.8 (GPIO6)
- new net: JP112.2 (B), JP113.1 (A), U129.26 (~{IRQ})
- new net: J124.1 (DAT2), R225.2
- new net: R192.2, R193.2, U148.13 (GPIO10)
- new net: R195.2, U148.11 (GPIO8)
- new net: R194.2, U148.12 (GPIO9)
- new net: R200.2, R206.2, R207.2, U148.14 (GPIO11)
- new net: R208.2, U148.15 (GPIO12)
- new net: R204.2, U148.16 (GPIO13)
- new net: R203.2, U148.17 (GPIO14)
- new net: R201.2, R202.2, U148.18 (GPIO15)
- new net: R182.2, R183.2, R190.2, U148.2 (GPIO0)
- new net: C135.1, U148.20 (XIN), Y101.3
- new net: R180.2, U148.21 (XOUT)
- new net: R181.2, SW104.2 (B), U148.26 (RUN)
- new net: R209.2, U148.27 (GPIO16)
- new net: R210.2, U148.28 (GPIO17)
- new net: R184.2, U148.3 (GPIO1)
- new net: R186.2, U148.4 (GPIO2)
- new net: R179.2, U148.46 (USB_DM)
- new net: R187.2, U148.5 (GPIO3)
- new net: U148.51 (QSPI_SD3), U150.7 (IO3)
- new net: U148.52 (QSPI_SCLK), U150.6 (CLK)
- new net: U148.53 (QSPI_SD0), U150.5 (DI(IO0))
- new net: U148.54 (QSPI_SD2), U150.3 (IO2)
- new net: U148.55 (QSPI_SD1), U150.2 (DO(IO1))
- new net: R176.2, R177.2, U148.56 (QSPI_SS), U150.1 (~{CS})
- new net: R188.2, R189.2, U148.6 (GPIO4)
- new net: R199.2, U148.9 (GPIO7)
- new net: Q102.1 (G), R216.2, R217.2
- new net: C136.1, R180.1, Y101.1
- new net: R176.1, SW103.2 (B)
- new net: D121.2 (A), R218.2
- new net: R190.1, SW105.1 (A)
- new net: JP107.1 (A), U130.14 (~{Y1})
- new net: JP106.1 (A), U130.15 (~{Y0})
- new net: R184.1, R185.2
- new net: D120.1 (K), J123.1 (VBUS), Q102.3 (D)
- new net: R200.1, SW107.1 (A)
- new net: J121.B5 (CC2), R211.2
- new net: J124.8 (DAT1), R226.2
- new net: Q103.3 (D), R216.1
- new net: R196.2, R199.1
- new net: R205.2, R208.1
- new net: D122.2 (A), R220.2
- new net: Q103.1 (G), R219.2
- new net: Q101.1 (G), R215.1
- new net: JP110.2 (B), JP111.1 (A), U107.26 (~{IRQ})
- new net: BZ101.2 (-), Q101.3 (D)
- new net +1V1: C123.1, C124.1, C125.1, U148.23 (DVDD), U148.45 (VREG_VOUT), U148.50 (DVDD)
- new net +3V3: C121.1, C126.1, C127.1, C128.1, C129.1, C130.1, C131.1, C132.1, C133.1, C134.1, J124.4 (VDD), J125.2 (Pin_2), Q104.1 (G), Q105.1 (G), R177.1, R181.1, R213.1, R214.1, R221.1, R223.1, R225.1, R226.1, SW105.2 (B), SW106.2 (B), SW107.2 (B), U148.1 (IOVDD), U148.10 (IOVDD), U148.22 (IOVDD), U148.33 (IOVDD), U148.42 (IOVDD), U148.43 (ADC_AVDD), U148.44 (VREG_IN), U148.48 (USB_VDD), U148.49 (IOVDD), U149.2 (VO), U150.8 (VCC), U151.8 (VDD)
- new net BUZZER: R215.2, U151.2 (IO1)
- new net HSYNC: J122.13, R209.1
- new net RP_102: J125.7 (Pin_7), U151.3 (IO2)
- new net RP_103: J125.8 (Pin_8), U151.5 (IO3)
- new net RP_18: R213.2, U148.29 (GPIO18), U151.7 (SDA)
- new net RP_19: R214.2, U148.30 (GPIO19), U151.6 (SCL)
- new net RP_20: Q104.2 (S), R221.2, U148.31 (GPIO20)
- new net RP_21: Q105.2 (S), R223.2, U148.32 (GPIO21)
- new net RP_22: J125.3 (Pin_3), U148.34 (GPIO22)
- new net RP_23: J125.4 (Pin_4), U148.35 (GPIO23)
- new net RP_24: J125.5 (Pin_5), U148.36 (GPIO24)
- new net RP_25: R220.1, U148.37 (GPIO25)
- new net RP_26: J124.5 (CLK), U148.38 (GPIO26_ADC0)
- new net RP_27: J124.3 (CMD), U148.39 (GPIO27_ADC1)
- new net RP_28: J124.7 (DAT0), U148.40 (GPIO28_ADC2)
- new net RP_29: J125.6 (Pin_6), U148.41 (GPIO29_ADC3)
- new net RP_5: J124.2 (DAT3/CD), U148.7 (GPIO5)
- new net RP_RX: J126.2 (Pin_2), Q105.3 (D), R224.2
- new net RP_TX: J126.3 (Pin_3), Q104.3 (D), R222.2
- new net USB+: J121.A6 (D+), J121.B6 (D+), J123.3 (D+), R178.1
- new net USB-: J121.A7 (D-), J121.B7 (D-), J123.2 (D-), R179.1
- new net USB_PWR: R218.1, R219.1, U151.1 (IO0)
- new net VGA_B: J122.3, R201.1, R202.1, R203.1, R204.1, R205.1, R206.1, R207.1
- new net VGA_G: J122.2, R192.1, R193.1, R194.1, R195.1, R196.1, R197.1, R198.1
- new net VGA_R: J122.1, R182.1, R183.1, R185.1, R186.1, R187.1, R188.1, R189.1
- new net VSYNC: J122.14, R210.1
- no-connect marks 94 -> 101
Other:
- note added: "Address PORT 96@32 -> 7F60 - 7F7F"
- note added: "Hardware Monitor"
- note added: "RP2040 PicoTerm"
- note added: "Solder Bridge Standard ACIA1: Address PORT 16@4 -> 7F50 - 7F53 ACIA2: Address PORT 20@4 -Y 7F54 - 7F57"
- note added: "Solder Bridge switched ACIA1: Address PORT 24@4 -> 7F58 - 7F5B ACIA2: Address PORT 28@4 -Y 7F5C - 7F5F"
- note added: "VIA1-COMMS"
- note removed: "ACIA1"
- note removed: "ACIA1: Address PORT 16@4 -> 7F50 - 7F53 ACIA2: Address PORT 20@4 -Y 7F54 - 7F57"
- note removed: "ACIA2"
- note removed: "Address PORT 192@32 -> 7FC0 - 7FDF"
- title: Massively Overblown Bream-Computer with 6502/65816 -> Massively Overblown Dream-Computer with 6502/65816
- moved on the sheet: U104
