File: Hardware/overview_65xx.kicad_sch (KiCad schematic)
At the start: 296 parts, among them J101 ABORT, J103 SO/MX, J105 Cx, J106 CF Card, J107 Barrel_Jack, J108 DE9_Plug_MountingHoles, J109 Conn_01x08, J110 DE9_Plug_MountingHoles, J111 Conn_01x08, J113 P2B, J114 P2A, J115 P3A, J116 P3B, J117 Conn_02x20_Odd_Even, J118 Conn_02x22_Odd_Even, J119 IDE_VCC, J120 Clock_Sel, J121 USB_C_Receptacle_USB2.0_14P, J122 DE15_Receptacle_HighDensity_M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, J123 Keyboard, J124 Micro_SD_Card, J125 IOs, J126 UART, Q101 BSS138, Q102 BSS84, Q103 BSS138, Q104 BSS138, Q105 BSS138, SW101 SW_SPDT, SW102 RESET, SW103 BOOTSEL, SW104 RST, SW105 T1, SW106 T2, SW107 T3, U101 65C02 / 65816, U102 SST39SF040, U103 W65C22SxP, U104 W65C22SxP, U105 6525, U106 6525, U107 6551, U108 W65C22SxP, U109 AS6C4008-55PCN, U110 CY62256-70PC, U111 74HC688, U112 74HC00, U113 74154, U114 74HC04, U115 6520, U116 74HC00, U117 74LS20, U118 74HC138, U119 8580, U120 AS6C4008-55PCN, U121 74HC00, U122 74HCT74, U123 74LS32, U124 74HC00, U125 MAX232, U126 MAX232, U127 MAX232, U128 MAX232, U129 6551, U130 74HC138, U131 74HC00, U132 74AHCT04, U133 74LS393, U134 74HC02, U135 74AHC04, U136 GAL16V8, U137 SA39-11EWA, U138 SA39-11EWA, U139 GAL16V8, U140 SA39-11EWA, U141 GAL16V8, U142 SA39-11EWA, U143 GAL16V8, U144 SA39-11EWA, U145 GAL16V8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

Commit message: ROM and CPU Card
Parts:
- added BT1: CR2032, symbol Device:Battery_Cell
- added R1, R2: 1k, symbol Device:R
- added U1: DS1501YZ, symbol 6502:DS1501YZ
- added U2, U3: 74HC00, symbol 74xx:74HC00
- added Y1: G33270007, Crystal:Crystal_SMD_FrontierElectronics_FM206, symbol Device:Crystal_GND3
Connections:
- net +5V: now also R1.1, R2.1, U1.28 (VCC)
- net A0: now also U1.6 (A0)
- net A1: now also U1.7 (A1)
- net A2: now also U1.8 (A2)
- net A3: now also U1.9 (A3)
- net CLK: now also U2.2, U3.1
- net D0: now also U1.11 (D0)
- net D1: now also U1.12 (D1)
- net D2: now also U1.13 (D2)
- net D3: now also U1.15 (D3)
- net D4: now also U1.16 (D4)
- net D5: now also U1.17 (D5)
- net D6: now also U1.18 (D6)
- net D7: now also U1.19 (D7)
- net GND: now also BT1.2 (-), U1.10 (A4), U1.14 (GND), U1.21 (GND), U1.26 (V_{BAUX}), Y1.3
- net PORT_160: now also U2.1
- net RAM0: now also U120.3 (A14)
- net RAM1: now also U120.31 (A15)
- net RAM2: now also U120.2 (A16)
- net RAM3: now also U120.30 (A17)
- net RAM4: now also U120.1 (A18)
- net ROM0: no longer U120.3 (A14)
- net ROM1: no longer U120.31 (A15)
- net ROM2: no longer U120.2 (A16)
- net ROM3: no longer U120.30 (A17)
- net ROM4: no longer U120.1 (A18)
- net R/~{W}: now also U1.27 (~{WE})
- net ~{IRQ_0.4}: now also U1.5 (~{IRQ})
- net ~{PAGE_RAM}: now also U3.2; no longer JP104.2 (B), U120.22 (CE#)
- net ~{RES}: now also U1.4 (~{RESET})
- new net: R2.2, U1.1 (~{PWR})
- new net: U1.2 (X1), Y1.1
- new net: U1.20 (~{CE}), U1.22 (~{OE}), U2.3
- new net: R1.2, U1.24 (~{KS})
- new net: BT1.1 (+), U1.25 (V_{BAT})
- new net: U1.3 (X2), Y1.2
- new net: JP104.2 (B), U120.22 (CE#), U3.3
- no-connect marks 101 -> 102
Other:
- note added: "Address PORT 160@16 -> BFA0 - BFAF"
- note added: "RTC"

Commit message: module update
Parts:
- added J1: Bus_PCI_6502, Connector_PCBEdge:BUS_PCI, symbol 6502:Bus_PCI_6502
Connections:
- net +5V: now also J1.A14 (5V), J1.A22 (5V), J1.A36 (5V), J1.A47 (5V), J1.B14 (5V), J1.B22 (5V), J1.B36 (5V), J1.B47 (5V)
- net +9V: now also J1.A49 (9V), J1.B49 (9V)
- net A0: now also J1.B2 (A0)
- net A1: now also J1.A2 (A1)
- net A10: now also J1.B9 (A10)
- net A11: now also J1.A9 (A11)
- net A12: now also J1.B11 (A12)
- net A13: now also J1.A11 (A13)
- net A14: now also J1.B12 (A14)
- net A15: now also J1.A12 (A15)
- net A2: now also J1.B3 (A2)
- net A3: now also J1.A3
- net A4: now also J1.B5 (A4)
- net A5: now also J1.A5
- net A6: now also J1.B6 (A6)
- net A7: now also J1.A6 (A7)
- net A8: now also J1.B8 (A8)
- net A9: now also J1.A8 (A9)
- net CLK: now also J1.B44 (CLK)
- net D0: now also J1.B16 (D0)
- net D1: now also J1.A16 (D1)
- net D2: now also J1.B17 (D2)
- net D3: now also J1.A17 (D3)
- net D4: now also J1.B19 (D4)
- net D5: now also J1.A19 (D5)
- net D6: now also J1.B20 (D6)
- net D7: now also J1.A20 (D7)
- net E: now also J1.A45 (E)
- net GND: now also J1.A1 (GND), J1.A10 (GND), J1.A13 (GND), J1.A15 (GND), J1.A18 (GND), J1.A21 (GND), J1.A23 (GND), J1.A26 (GND), J1.A35 (GND), J1.A37 (GND), J1.A4 (GND), J1.A40 (GND), J1.A43 (GND), J1.A44 (GND), J1.A46 (GND), J1.A48 (GND), J1.A52 (GND), J1.A57 (GND), J1.A62 (GND), J1.A7 (GND), J1.B1 (GND), J1.B10 (GND), J1.B13 (GND), J1.B15 (GND), J1.B18 (GND), J1.B21 (GND), J1.B23 (GND), J1.B26 (GND), J1.B35 (GND), J1.B37 (GND), J1.B4 (GND), J1.B40 (GND), J1.B43 (GND), J1.B45 (GND), J1.B48 (GND), J1.B52 (GND), J1.B57 (GND), J1.B62 (GND), J1.B7 (GND)
- net M/X: now also J1.B46 (M/~{X})
- net PAGE: now also J1.B34 (PAGE_ROM)
- net R/~{W}: now also J1.B42 (R/~{W})
- net ~{H_RAM}: now also J1.B25 (~{H_RAM})
- net ~{IO}: now also J1.A24 (~{IO})
- net ~{IRQ_0.0}: now also J1.A27 (~{IRQ_0.0})
- net ~{IRQ_0.1}: now also J1.A28 (~{IRQ_0.1})
- net ~{IRQ_0.2}: now also J1.A29 (~{IRQ_0.2})
- net ~{IRQ_0.3}: now also J1.A30 (~{IRQ_0.3})
- net ~{IRQ_0.4}: now also J1.A31 (~{IRQ_0.4})
- net ~{IRQ_0.5}: now also J1.A32 (~{IRQ_0.5})
- net ~{IRQ_0.6}: now also J1.A33 (~{IRQ_0.6})
- net ~{IRQ_0.7}: now also J1.A34 (~{IRQ_0.7})
- net ~{IRQ_0}: now also J1.B28 (~{IRQ_0})
- net ~{IRQ_1}: now also J1.B29 (~{IRQ_1})
- net ~{IRQ_2}: now also J1.B30 (~{IRQ_2})
- net ~{IRQ_3}: now also J1.B31 (~{IRQ_3})
- net ~{IRQ_4}: now also J1.B32 (~{IRQ_4})
- net ~{IRQ}: now also J1.B27 (~{IRQ})
- net ~{L_RAM}: now also J1.B24 (~{L_RAM})
- net ~{ML}: now also J1.B39 (~{ML})
- net ~{NMI}: now also J1.B33 (~{NMI})
- net ~{RES}: now also J1.B41 (~{RES})
- net ~{ROM}: now also J1.A25 (~{ROM})
- net ~{VP}: now also J1.B38 (~{VP})
- new net RAM_0: J1.A53 (RAM0)
- new net RAM_1: J1.A54 (RAM1)
- new net RAM_2: J1.A55 (RAM2)
- new net RAM_3: J1.A56 (RAM3)
- new net RAM_4: J1.A58 (RAM4)
- new net RAM_5: J1.A59 (RAM5)
- new net RAM_6: J1.A60 (RAM6)
- new net RAM_7: J1.A61 (RAM7)
- new net ROM_0: J1.B53 (ROM0)
- new net ROM_1: J1.B54 (ROM1)
- new net ROM_2: J1.B55 (ROM2)
- new net ROM_3: J1.B56 (ROM3)
- new net ROM_4: J1.B58 (ROM4)
- new net ROM_5: J1.B59 (ROM5)
- new net ROM_6: J1.B60 (ROM6)
- new net ROM_7: J1.B61 (ROM7)
- new net SYNC_VPA: J1.A38 (Sync/VPA)
- new net ~{BE}: J1.A42 (~{BE})
- new net ~{RDY}: J1.A41 (~{RDY})
- new net Ø2/VDA: J1.A39 (Ø2/VDA)
