File: Hardware/modules/Address_Decode/Address_Decode.kicad_pcb (KiCad board)
At the start: 4 copper layers, 83.3 x 68.2 mm, 28 parts, among them J1 Bus_PCI_6502, J2 Clock_Sel, J3 Conn_01x08, SW1 Manual_Clock, U1 74HC14, U2 74HC00, U3 74LS20, U4 DS1501YZ, U5 74LS393, U6 74HC138, U7 74HC688, X1 8MHz, Y1 G33270007

Commit message: Update Module Files and Readme
Parts:
- added G***: LOGO, Eigene:logo, F.Cu at (181.1, 49.0)
- added REF**: WEEE-Logo_5.6x8mm_SilkScreen, Symbol:WEEE-Logo_5.6x8mm_SilkScreen, F.Cu at (181.4, 68.8)
- added REF**: ESD-Logo_8.9x8mm_SilkScreen, Symbol:ESD-Logo_8.9x8mm_SilkScreen, F.Cu at (181.1, 59.7)
- added REF**: OSHW-Logo2_9.8x8mm_SilkScreen, Symbol:OSHW-Logo2_9.8x8mm_SilkScreen, F.Cu at (181.4, 77.7)
- added Ref**: Val**, Eigene:ladder_4, F.Cu at (144.5, 35.6)
Other:
- board text added: "125"
- board text added: "1M"
- board text added: "1k"
- board text added: "250"
- board text added: "2M"
- board text added: "4M"
- board text added: "500"
- board text added: "500k"
- board text added: "62.5"
- board text added: "8M"
- board text added: "MAN"
- board text added: "SY65 Clock ADDR RTC"
