File: Hardware/modules/Bus_Card/Bus_Card.kicad_sch (KiCad schematic)
At the start: 19 parts, among them J1 DC In, SW1 RESET, SW2 NMI, U1 SY317, U2 SY317

Commit message: Hardware Review Pt. 1 fix Address Decoding for Strobe Generators add bulk capacitance to every board fix wiring of Prototyping Board
Parts:
- SW1, SW2: footprint Button_Switch_SMD:SW_Push_1P1T_XKB_TS-1187A -> Button_Switch_THT:SW_PUSH_6mm
Changed lines of the file:
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@@
 			)
 		)
-		(property "Footprint" "Button_Switch_SMD:SW_Push_1P1T_XKB_TS-1187A"
+		(property "Footprint" "Button_Switch_THT:SW_PUSH_6mm"
 			(at 275.59 229.87 0)
 			(effects
@@
 			)
 		)
-		(property "Footprint" "Button_Switch_SMD:SW_Push_1P1T_XKB_TS-1187A"
+		(property "Footprint" "Button_Switch_THT:SW_PUSH_6mm"
 			(at 275.59 222.25 0)
 			(effects
